File: extractor-smd/extractor-smd.sch (KiCad schematic (older format))
At the start: 17 parts, among them J1 Conn_Coaxial, J2 Screw_Terminal_01x02, J3 Conn_Coaxial

Commit message: Add files via upload
Updated RF paths to 2.5mm with
Other:
- moved on the sheet: C1, C2, C3, C4, C5, C6, D1, H1, H2, H3, H4, J1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
