File: extractor-smd/bias-t-extractor-smd.kicad_pcb (KiCad board)
At the start: 2 copper layers, 42 x 56 mm, 17 parts, among them J1 Conn_Coaxial, J2 Screw_Terminal_01x02, J3 Conn_Coaxial

Commit message: updated files and BOM's .
Parts:
- C1, C5, C6: value CAP CER 10000PF 2KV X7R 1812 -> 0.01uF
- L1, L2: value 744762210A -> SRU8045A-101Y; footprint Inductor_SMD:L_1008_2520Metric -> Inductor_SMD:L_Bourns-SRU8045A-101Y_8.0x8.0mm
- moved D1 6.67 mm to (58.4, 58.5)
- moved J2 6.67 mm to (47.5, 60.2)
- moved LA1 6.67 mm to (69.5, 57.2)
- moved C2 4.50 mm to (50.1, 51.5)
- moved C3 4.50 mm to (65.6, 51.0)
- moved C4 4.50 mm to (57.8, 51.0)
- moved L2 2.35 mm to (65.0, 36.1)
- moved L1 1.86 mm to (51.1, 44.0)
Connections:
- net /DC+ renamed Net-(C2-Pad1)
- net /DC-GND renamed /GND
Routing:
- net /GND: track 75.0 -> 14.0 mm
- net Net-(C2-Pad1): track 61.2 -> 53.7 mm
- net /RF+DC: track 26.5 -> 24.4 mm
- net /RF-GND: track 33.5 -> 31.6 mm
Other:
- board text added: "COAX SHIELD"
- board text added: "RF OUT"
- board text added: "RF+DC IN"

Commit message: Add files via upload
Updated RF paths to 2.5mm with
Routing:
- net /RF+DC: track 24.4 -> 25.6 mm
- net /RF-GND: track 31.6 -> 32.4 mm
Other:
- net class RF: trace_width 0.7 -> 2.5
- net class RF-GND: trace_width 0.7 -> 2.5

Commit message: Add files via upload
Other:
- board text added: "DC OUT"
