File: injector-smd/bias-t-injector-smd.kicad_pcb (KiCad board)
At the start: 2 copper layers, 42 x 56 mm, 18 parts, among them J1 Conn_Coaxial, J2 Screw_Terminal_01x02, J3 Conn_Coaxial

Commit message: updated files and BOM's .
Parts:
- C1, C5, C6: value CAP CER 10000PF 2KV X7R 1812 -> 0.01uF
- L1, L2: value 744762210A -> SRU8045A-101Y; footprint Inductor_SMD:L_1008_2520Metric -> Inductor_SMD:L_Bourns-SRU8045A-101Y_8.0x8.0mm
- moved C4 4.67 mm to (56.5, 51.0)
- moved C3 4.50 mm to (65.6, 51.0)
- moved C2 4.31 mm to (48.5, 51.0)
- moved D1 4.00 mm to (56.9, 56.0)
- moved LA1 3.75 mm to (68.0, 54.5)
- moved F1 3.54 mm to (62.5, 65.0)
- moved J2 3.25 mm to (46.0, 57.0)
- moved L2 2.35 mm to (65.0, 36.1)
- moved L1 1.50 mm to (50.0, 44.0)
Connections:
- net /DC+ renamed Net-(C2-Pad1)
- net /DC-GND renamed /GND
Routing:
- net /GND: track 78.7 -> 25.3 mm
- net Net-(C2-Pad1): track 44.6 -> 50.5 mm, vias 0 -> 4
- net Net-(D1-Pad1): track 21.3 -> 18.7 mm
- net /RF+DC: track 26.5 -> 24.4 mm
- net /RF-GND: track 33.5 -> 31.6 mm
Other:
- board text added: "COAX SHIELD"
- board text added: "RF OUT"
- board text added: "RF+DC IN"

Commit message: Add files via upload
Updated RF paths to 2.5mm with.
Routing:
- net /RF+DC: track 24.4 -> 25.7 mm
- net /RF-GND: track 31.6 -> 32.2 mm
Other:
- net class RF: trace_width 0.7 -> 2.5
- net class RF-GND: trace_width 0.7 -> 2.5

Commit message: Add files via upload
Other:
- board text added: "DC IN"
- board text added: "RF IN"
- board text added: "RF+DC OUT"
- board text removed: "RF OUT"
- board text removed: "RF+DC IN"
